File: Soldering iron 936A + t12 compatible.kicad_pcb (KiCad board)
At the start: 2 copper layers, 97 x 67 mm, 103 parts, among them J1 DC INPUT, J10 Conn_01x01_Socket, J11 Conn_01x01_Socket, J3 AC input, J4 output_connector, J5 mosfet_driver_future_backup, J6 OLED, J7 USB C BREAKOUT BOARD, J8 TOP LEFT, Q1 IRF9540N, Q2 BC547, SW1 RotaryEncoder_Switch, U1 LM2596S-ADJ, U2 LM358, U4 HUSB238, U8 INA219AxD

Commit message: re working on layout now
Parts:
- removed C19: 1000uF, Capacitor_THT:CP_Radial_D16.0mm_P7.50mm
- removed J10, J11: Conn_01x01_Socket, Connector_PinHeader_2.54mm:PinHeader_1x01_P2.54mm_Vertical
- removed J5: mosfet_driver_future_backup, Connector_PinHeader_2.54mm:PinHeader_1x06_P2.54mm_Vertical
- removed J8: TOP LEFT, Connector_PinHeader_2.54mm:PinHeader_1x02_P2.54mm_Vertical_SMD_Pin1Left
- added F1: Fuse, Fuse:Fuse_1206_3216Metric_Pad1.42x1.75mm_HandSolder, B.Cu at (209.6, 100.0)
- added R35: 1M, Resistor_SMD:R_1206_3216Metric_Pad1.30x1.75mm_HandSolder, B.Cu at (209.6, 97.7)
- added R36: 50K, Resistor_SMD:R_1206_3216Metric_Pad1.30x1.75mm_HandSolder, B.Cu at (212.3, 104.6)
- added R37: 10k, Resistor_SMD:R_1206_3216Metric_Pad1.30x1.75mm_HandSolder, F.Cu at (208.7, 83.0)
- added U3: HCPL-3700, Package_DIP:DIP-8_W7.62mm, F.Cu at (201.9, 102.3)
Connections:
- A2 pad 12: /LEAK_ERR -> unconnected-(A2-GPIO9-Pad12)
- A2 pad 26: /PWM1 -> /LEAK_ERR
- J4 pad 6: Earth -> Net-(J4-Pin_6)
Routing:
- net /PWM: track 41.5 -> 82.9 mm, vias 2 -> 1
- net Net-(J4-Pin_6): track 0.00 -> 27.2 mm
- net Net-(Q2-C): track 68.9 -> 48.8 mm
- net /PWM1: track 18.3 -> 0.00 mm, vias 1 -> 0
- net Earth: track 27.5 -> 10.5 mm
- net /LEAK_ERR: track 0.00 -> 13.0 mm, vias 0 -> 1
- net /VIN: track 120.8 -> 111.3 mm
- net GND: track 108.1 -> 103.1 mm, vias 73 -> 74
- net /ENCODER S: track 106.1 -> 110.6 mm
- net Net-(R36-Pad1): track 0.00 -> 2.84 mm
