File: Soldering iron 936A + t12 compatible.kicad_sch (KiCad schematic)
At the start: 104 parts, among them J1 DC INPUT, J10 Conn_01x01_Socket, J11 Conn_01x01_Socket, J3 AC input, J4 output_connector, J5 mosfet_driver_future_backup, J6 OLED, J7 USB C BREAKOUT BOARD, J8 TOP LEFT, Q1 IRF9540N, Q2 BC547, SW1 RotaryEncoder_Switch, U1 LM2596S-ADJ, U2 LM358, U4 HUSB238, U8 INA219AxD

Commit message: re working on layout now
Parts:
- removed C19: 1000uF, Capacitor_THT:CP_Radial_D16.0mm_P7.50mm, symbol Device:C_Polarized
- removed J10, J11: Conn_01x01_Socket, Connector_PinHeader_2.54mm:PinHeader_1x01_P2.54mm_Vertical, symbol Connector:Conn_01x01_Socket
- removed J5: mosfet_driver_future_backup, Connector_PinHeader_2.54mm:PinHeader_1x06_P2.54mm_Vertical, symbol Connector:Conn_01x06_Pin
- removed J8: TOP LEFT, Connector_PinHeader_2.54mm:PinHeader_1x02_P2.54mm_Vertical_SMD_Pin1Left, symbol Connector:Conn_01x02_Socket
- added F1: Fuse, Fuse:Fuse_1206_3216Metric_Pad1.42x1.75mm_HandSolder, symbol Device:Fuse
- added R35: 1M, Resistor_SMD:R_1206_3216Metric_Pad1.30x1.75mm_HandSolder, symbol Device:R
- added R36: 50K, Resistor_SMD:R_1206_3216Metric_Pad1.30x1.75mm_HandSolder, symbol Device:R
- added R37: 10k, Resistor_SMD:R_1206_3216Metric_Pad1.30x1.75mm_HandSolder, symbol Device:R
- added U3: HCPL-3700, Package_DIP:DIP-8_W7.62mm, symbol Isolator:HCPL-261A
Connections:
- net +3.3V: now also R37.2, U3.8 (VCC)
- net Earth: now also F1.1, R35.2, R36.2; no longer J4.6 (Pin_6)
- net GND: now also U3.5 (GND)
- net LEAK_ERR: now also R37.1, U3.6 (VO)
- new net: R36.1, U3.1 (AC)
- new net TIP_EARTH: F1.2, J4.6 (Pin_6), R35.1, U3.4 (AC)
- no-connect marks 6 -> 4
